File: JGA25-370B_with_l289_driver_2_channel.kicad_pcb (KiCad board)
At the start: 2 copper layers, 152.4 x 99.1 mm, 36 parts, among them J1 Power 12 V, J2 Output 1, J3 Encoder 1, J4 Encoder 1 Power 3.3V, J5 Output 2, J6 Encoder 2, J7 Encoder 2 Power 3.3V, J8 Power 5 V, Q1 2N7002, Q2 2N7002, Q3 2N7002, SW1 forward_device_1, SW2 backward_device_1, SW3 stop_device_1, SW4 forward_device_2, SW5 backward_device_2, SW6 stop_device_2, SW7 to_reset_all, U1 L289N_shield, U2 ESP32-S2-DevKitM

Commit message: fix nets
Parts:
- added C1: C, Capacitor_SMD:C_1206_3216Metric, B.Cu at (197.1, 94.9)
- added C10: C_Polarized, Capacitor_THT:CP_Radial_D10.0mm_P2.50mm, F.Cu at (195.6, 40.6)
- added C2: C, Capacitor_SMD:C_1206_3216Metric, B.Cu at (197.1, 98.2)
- added C3: C_Polarized, Capacitor_THT:CP_Radial_D10.0mm_P2.50mm, F.Cu at (182.9, 63.5)
- added C4: c=C_Polarized, Capacitor_THT:CP_Radial_D10.0mm_P2.50mm, F.Cu at (195.6, 63.5)
- added C5: C, Capacitor_THT:C_Disc_D9.0mm_W5.0mm_P5.00mm, F.Cu at (180.3, 81.4)
- added C6: C, Capacitor_THT:C_Disc_D9.0mm_W5.0mm_P5.00mm, F.Cu at (114.3, 78.8)
- added C7: C_Polarized, Capacitor_THT:CP_Radial_D10.0mm_P2.50mm, F.Cu at (182.9, 40.6)
- added C8: C, Capacitor_SMD:C_1206_3216Metric, B.Cu at (197.1, 101.6)
- added C9: C, Capacitor_SMD:C_1206_3216Metric, B.Cu at (197.1, 105.0)
- added R10: 330, Resistor_SMD:R_1206_3216Metric, F.Cu at (86.1, 93.8)
- added R14: 10k, Resistor_SMD:R_1206_3216Metric, F.Cu at (86.1, 97.1)
- added R14: 330, Resistor_SMD:R_1206_3216Metric, B.Cu at (197.1, 116.8)
- added R5: 10k, Resistor_SMD:R_1206_3216Metric, F.Cu at (86.1, 87.2)
- added R6: 4.7k, Resistor_SMD:R_1206_3216Metric, F.Cu at (86.1, 90.5)
- added SW4: forward_device_2, Button_Switch_THT:SW_PUSH_6mm_H4.3mm, F.Cu at (74.8, 87.6)
- added SW5: backward_device_2, Button_Switch_THT:SW_PUSH_6mm_H4.3mm, F.Cu at (74.8, 96.2)
- added SW6: stop_device_2, Button_Switch_THT:SW_PUSH_6mm_H4.3mm, F.Cu at (74.8, 104.7)
- added SW8: undef, Button_Switch_THT:SW_PUSH_6mm_H4.3mm, F.Cu at (57.7, 84.1)
- added U3: LM1117T-5.0, Package_TO_SOT_THT:TO-220-3_Vertical, F.Cu at (188.0, 33.0)
- added U4: LM1117T-3.3, Package_TO_SOT_THT:TO-220-3_Vertical, F.Cu at (188.0, 53.3)
- R4: value 330 -> 4.7k
- R7: value 330 -> 2.2k
- R8, R9: value 330 -> 10k
- SW7: value to_reset_all -> undef
- U2: value ESP32-S2-DevKitM -> ESP32-DevKitC; footprint PCM_Espressif:ESP32-S2-DevKitM -> PCM_Espressif:ESP32-DevKitC
- moved D1 160.2 mm to (55.9, 111.8)
- moved D3 143.1 mm to (55.9, 104.1)
- moved SW4 124.6 mm to (57.7, 53.6)
- moved SW5 124.5 mm to (57.7, 61.2)
- moved SW6 124.5 mm to (57.7, 68.9)
- moved D2 123.9 mm to (55.9, 96.5)
- moved SW7 117.0 mm to (57.7, 76.5)
- moved SW3 109.1 mm to (57.7, 46.0)
- moved SW2 108.6 mm to (57.7, 38.4)
- moved SW1 108.2 mm to (64.2, 35.3)
- moved R10 78.4 mm to (98.5, 108.2)
- moved R6 78.4 mm to (98.5, 95.0)
- moved R7 78.4 mm to (98.5, 98.3)
- moved R8 78.4 mm to (98.5, 101.6)
- moved R9 78.4 mm to (98.5, 104.9)
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Connections:
- R4 pad 1: Net-(R10-Pad1) -> control_curtains_2
- R4 pad 2: sw_back_1 -> Net-(R4-Pad2)
- R6 pad 2: reset -> undef1
- R7 pad 1: Net-(R10-Pad1) -> Net-(R7-Pad1)
- R7 pad 2: sw_forw_1 -> control_curtains_2
- R8 pad 1: Net-(R10-Pad1) -> control_curtains_2
- R8 pad 2: sw_forw_2 -> GND
- R9 pad 1: Net-(R10-Pad1) -> Net-(R9-Pad1)
- R9 pad 2: sw_back_2 -> control_curtains_2
- SW1 pad 1: sw_forw_1 -> 3.3V
- SW1 pad 2: GND -> Net-(R9-Pad1)
- SW2 pad 1: sw_back_1 -> 3.3V
- SW2 pad 2: GND -> Net-(R4-Pad2)
- SW3 pad 1: sw_stop_1 -> 3.3V
- SW3 pad 2: GND -> Net-(R7-Pad1)
- SW4 pad 2: GND -> Net-(SW4-Pad2)
- SW5 pad 2: GND -> Net-(SW4-Pad2)
- SW6 pad 2: GND -> Net-(SW4-Pad2)
- SW7 pad 1: reset -> undef1
- U2 pad 1: 3.3V -> 5V
- U2 pad 10: unconnected-(U2-GPIO8/TOUCH8/ADC1_CH7-Pad10) -> motor_1_state
- U2 pad 11: Enc1_1 -> moto_2_state
- U2 pad 12: Enc1_2 -> Enc2_2
- U2 pad 13: Enc2_1 -> unconnected-(U2-MTDI/GPIO12/ADC2_CH5-Pad13)
- U2 pad 14: Enc2_2 -> GND
- U2 pad 15: wifi_state -> Enc2_1
- U2 pad 16: motor_1_state -> unconnected-(U2-SD_DATA2/GPIO9-Pad16)
- U2 pad 19: moto_2_state -> 3.3V
- U2 pad 20: 5V -> unconnected-(U2-SD_CLK/GPIO6-Pad20)
- U2 pad 21: GND -> unconnected-(U2-SD_DATA0/GPIO7-Pad21)
- U2 pad 25: sw_forw_1 -> unconnected-(U2-GPIO0/BOOT/ADC2_CH1-Pad25)
- U2 pad 26: unconnected-(U2-GPIO26-Pad26) -> PWM2
- U2 pad 27: sw_back_1 -> Enc1_2
- U2 pad 28: sw_stop_1 -> Enc1_1
- U2 pad 29: sw_forw_2 -> unconnected-(U2-GPIO5-Pad29)
- U2 pad 3: PWM1 -> unconnected-(U2-SENSOR_VP/GPIO36/ADC1_CH0-Pad3)
- U2 pad 30: sw_back_2 -> In4
- U2 pad 31: sw_stop_2 -> In3
- U2 pad 32: reset -> GND
- U2 pad 33: unconnected-(U2-MTCK/JTAG/GPIO39-Pad33) -> In2
- U2 pad 36: unconnected-(U2-MTMS/JTAG/GPIO42-Pad36) -> In1
- U2 pad 37: unconnected-(U2-U0TXD/GPIO43/CLK_OUT1-Pad37) -> PWM1
- U2 pad 38: unconnected-(U2-U0RXD/GPIO44/CLK_OUT2-Pad38) -> GND
- U2 pad 4: In1 -> unconnected-(U2-SENSOR_VN/GPIO39/ADC1_CH3-Pad4)
- U2 pad 5: In2 -> unconnected-(U2-VDET_1/GPIO34/ADC1_CH6-Pad5)
- U2 pad 6: In3 -> unconnected-(U2-VDET_2/GPIO35/ADC1_CH7-Pad6)
- U2 pad 7: In4 -> control_curtains_1
- U2 pad 8: PWM2 -> control_curtains_2
- U2 pad 9: unconnected-(U2-GPIO7/TOUCH7/ADC1_CH6-Pad9) -> wifi_state

Commit message: ready for order
Parts:
- removed C10, C7: C_Polarized, Capacitor_THT:CP_Radial_D10.0mm_P2.50mm
- removed C5, C6: C, Capacitor_THT:C_Disc_D9.0mm_W5.0mm_P5.00mm
- removed C8, C9: C, Capacitor_SMD:C_1206_3216Metric
- removed J7: Encoder 2 Power 3.3V, Connector_JST:JST_EH_B2B-EH-A_1x02_P2.50mm_Vertical
- removed J8: Power 5 V, Connector_JST:JST_EH_B2B-EH-A_1x02_P2.50mm_Vertical
- removed the R10 at (86.1, 93.8)
- removed the R10 at (98.5, 108.2)
- removed the R14 at (86.1, 97.1)
- removed the R14 at (197.1, 116.8)
- removed the R5 at (86.1, 87.2)
- removed the R5 at (104.1, 108.2)
- removed the R6 at (86.1, 90.5)
- removed the R6 at (98.5, 95.0)
- removed the SW4 at (74.8, 87.6)
- removed the SW4 at (57.7, 53.6)
- removed the SW5 at (74.8, 96.2)
- removed the SW5 at (57.7, 61.2)
- removed the SW6 at (57.7, 68.9)
- removed the SW6 at (74.8, 104.7)
- removed SW7, SW8: undef, Button_Switch_THT:SW_PUSH_6mm_H4.3mm
- removed U3: LM1117T-5.0, Package_TO_SOT_THT:TO-220-3_Vertical
- removed U4: LM1117T-3.3, Package_TO_SOT_THT:TO-220-3_Vertical
- added PS1: Step_Down_3.3v_3A, Converter_DCDC:Converter_DCDC_3A_step_down_3.3v, F.Cu at (123.2, 91.2)
- added R10: 4.7k, Resistor_SMD:R_1206_3216Metric, B.Cu at (64.1, 69.6)
- added R14: 330, Resistor_SMD:R_1206_3216Metric, B.Cu at (62.0, 91.7)
- added R5: 10k, Resistor_SMD:R_1206_3216Metric, B.Cu at (63.8, 30.7)
- added R6: 330, Resistor_SMD:R_1206_3216Metric, B.Cu at (62.2, 85.3)
- added SW4: forward_device_2, Button_Switch_THT:SW_PUSH_6mm_H4.3mm, F.Cu at (53.5, 56.5)
- added SW5: backward_device_2, Button_Switch_THT:SW_PUSH_6mm_H4.3mm, F.Cu at (53.5, 65.0)
- added SW6: stop_device_2, Button_Switch_THT:SW_PUSH_6mm_H4.3mm, F.Cu at (53.5, 73.5)
- C1, C2: footprint Capacitor_SMD:C_1206_3216Metric -> Capacitor_THT:C_Disc_D9.0mm_W5.0mm_P5.00mm; moved to F.Cu
- D2: value Motor 1 Working -> Motor 2 Working
- D3: value Motor 2 Working -> Motor 1 Working
- J1: value Power 12 V -> Conn_01x03; footprint Connector_JST:JST_EH_B2B-EH-A_1x02_P2.50mm_Vertical -> TerminalBlock_MetzConnect:TerminalBlock_MetzConnect_Type101_RT01603HBWC_1x03_P5.08mm_Horizontal
- J2: value Output 1 -> Conn_01x03; footprint Connector_JST:JST_EH_B2B-EH-A_1x02_P2.50mm_Vertical -> TerminalBlock_MetzConnect:TerminalBlock_MetzConnect_Type101_RT01603HBWC_1x03_P5.08mm_Horizontal
- J3: value Encoder 1 -> Conn_01x03; footprint Connector_JST:JST_EH_B2B-EH-A_1x02_P2.50mm_Vertical -> TerminalBlock_MetzConnect:TerminalBlock_MetzConnect_Type101_RT01603HBWC_1x03_P5.08mm_Horizontal
- J4: value Encoder 1 Power 3.3V -> Conn_01x03; footprint Connector_JST:JST_EH_B2B-EH-A_1x02_P2.50mm_Vertical -> TerminalBlock_MetzConnect:TerminalBlock_MetzConnect_Type101_RT01603HBWC_1x03_P5.08mm_Horizontal
- J5: value Output 2 -> Conn_01x04_Pin; footprint Connector_JST:JST_EH_B2B-EH-A_1x02_P2.50mm_Vertical -> Connector_PinHeader_2.54mm:PinHeader_1x04_P2.54mm_Vertical
- J6: value Encoder 2 -> Conn_01x04_Pin; footprint Connector_JST:JST_EH_B2B-EH-A_1x02_P2.50mm_Vertical -> Connector_PinHeader_2.54mm:PinHeader_1x04_P2.54mm_Vertical
- R12, R2: value 330 -> 10k
- R3: value 330 -> 4.7k
- R4: value 4.7k -> 2.2k
- R7: value 2.2k -> 330
- R8: value 10k -> 330
- U1: value L289N_shield -> ESP32-DevKitC; footprint Library:L298n_motor_driver_shield -> PCM_Espressif:ESP32-DevKitC
- U2: value ESP32-DevKitC -> L289N_shield; footprint PCM_Espressif:ESP32-DevKitC -> Library:L298n_motor_driver_shield
- moved C3 92.8 mm to (95.0, 93.2), turned to -90 degrees
- moved C1 77.5 mm to (120.7, 107.6)
- moved R2 74.8 mm to (63.8, 35.3), turned to 0 degrees
- moved J2 71.5 mm to (132.1, 115.0), turned to 0 degrees
- moved R3 70.3 mm to (63.8, 43.9)
- moved C4 68.1 mm to (134.6, 93.7), turned to -90 degrees
- moved J5 66.9 mm to (136.4, 84.1), turned to 90 degrees
- moved R4 66.1 mm to (63.8, 52.6), turned to 0 degrees
- moved R9 55.9 mm to (64.0, 61.0), turned to 0 degrees
- moved C2 55.6 mm to (142.2, 107.6)
- moved R12 50.9 mm to (64.0, 56.4)
- moved U1 48.9 mm to (73.7, 34.0)
- moved J1 45.0 mm to (115.6, 115.0), turned to 0 degrees
- moved R1 43.7 mm to (62.2, 82.9), turned to 180 degrees
- moved J6 40.1 mm to (103.6, 84.1), turned to 90 degrees
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Connections:
- C1 pad 1: 12V -> Output1_1
- C1 pad 2: GND -> Output1_2
- C2 pad 1: 5V -> Output2_1
- C2 pad 2: GND -> Output2_2
- C3 pad 1: 5V -> 3.3V
- D1 pad 1: GND -> Net-(D1-K)
- D1 pad 2: Net-(D1-A) -> 3.3V
- D2 pad 1: GND -> Net-(D2-K)
- D2 pad 2: Net-(D2-A) -> 3.3V
- D3 pad 1: GND -> Net-(D3-K)
- D3 pad 2: Net-(D3-A) -> 3.3V
- J1 pad 1: 12V -> Output1_2
- J1 pad 2: GND -> Output1_1
- J2 pad 1: Output1_1 -> 12V
- J2 pad 2: Output1_2 -> Output2_2
- J3 pad 1: Enc1_2 -> GND
- J4 pad 1: 3.3V -> Enc2_2
- J4 pad 2: GND -> Enc2_1
- J5 pad 1: Output2_1 -> 3.3V
- J5 pad 2: Output2_2 -> In3
- J6 pad 1: Enc2_1 -> 3.3V
- J6 pad 2: Enc2_2 -> Enc1_1
- Q1 pad 2: Net-(D1-A) -> Net-(Q1-S)
- Q1 pad 3: Net-(Q1-D) -> Net-(D1-K)
- Q2 pad 2: Net-(D2-A) -> Net-(Q2-S)
- Q2 pad 3: Net-(Q2-D) -> Net-(D2-K)
- Q3 pad 2: Net-(D3-A) -> Net-(Q3-S)
- Q3 pad 3: Net-(Q3-D) -> Net-(D3-K)
- R1 pad 1: Net-(R1-Pad1) -> wifi_state
- R1 pad 2: Net-(Q1-D) -> Net-(Q1-G)
- R11 pad 1: Net-(R1-Pad1) -> Net-(R11-Pad1)
- R11 pad 2: Net-(Q2-D) -> control_curtains_1
- R12 pad 1: moto_2_state -> control_curtains_1
- R12 pad 2: Net-(Q3-G) -> GND
- R13 pad 1: Net-(R1-Pad1) -> motor_1_state
- R13 pad 2: Net-(Q3-D) -> Net-(Q3-G)
- R2 pad 1: wifi_state -> Net-(R2-Pad1)
- R2 pad 2: Net-(Q1-G) -> control_curtains_2
- R3 pad 1: motor_1_state -> control_curtains_2
- R3 pad 2: Net-(Q2-G) -> Net-(R3-Pad2)
- R4 pad 1: control_curtains_2 -> Net-(R4-Pad1)
- R4 pad 2: Net-(R4-Pad2) -> control_curtains_2
- R7 pad 1: Net-(R7-Pad1) -> moto_2_state
- R7 pad 2: control_curtains_2 -> Net-(Q2-G)
- R8 pad 1: control_curtains_2 -> Net-(Q2-S)
- R9 pad 2: control_curtains_2 -> control_curtains_1
- SW1 pad 2: Net-(R9-Pad1) -> Net-(R2-Pad1)
- SW2 pad 2: Net-(R4-Pad2) -> Net-(R3-Pad2)
- SW3 pad 2: Net-(R7-Pad1) -> Net-(R4-Pad1)
- U1 pad 1: Output1_1 -> 3.3V
- U1 pad 10: In4 -> motor_1_state
- U1 pad 11: PWM2 -> moto_2_state
- U1 pad 12: Output2_2 -> Enc2_2
- U1 pad 13: Output2_1 -> unconnected-(U1-MTDI/GPIO12/ADC2_CH5-Pad13)
- U1 pad 2: Output1_2 -> unconnected-(U1-CHIP_PU-Pad2)
- U1 pad 3: GND -> unconnected-(U1-SENSOR_VP/GPIO36/ADC1_CH0-Pad3)
- U1 pad 4: 12V -> unconnected-(U1-SENSOR_VN/GPIO39/ADC1_CH3-Pad4)
- U1 pad 6: PWM1 -> unconnected-(U1-VDET_2/GPIO35/ADC1_CH7-Pad6)
- U1 pad 7: In1 -> control_curtains_2
- U1 pad 8: In2 -> control_curtains_1
- U1 pad 9: In3 -> wifi_state
- U2 pad 1: 5V -> Output1_1
- U2 pad 10: motor_1_state -> In4
- U2 pad 11: moto_2_state -> PWM2
- U2 pad 12: Enc2_2 -> Output2_2
- U2 pad 13: unconnected-(U2-MTDI/GPIO12/ADC2_CH5-Pad13) -> Output2_1
- U2 pad 2: unconnected-(U2-CHIP_PU-Pad2) -> Output1_2
- U2 pad 3: unconnected-(U2-SENSOR_VP/GPIO36/ADC1_CH0-Pad3) -> GND
- U2 pad 4: unconnected-(U2-SENSOR_VN/GPIO39/ADC1_CH3-Pad4) -> 12V
- U2 pad 6: unconnected-(U2-VDET_2/GPIO35/ADC1_CH7-Pad6) -> PWM1
- U2 pad 7: control_curtains_1 -> In1
- U2 pad 8: control_curtains_2 -> In2
- U2 pad 9: wifi_state -> In3
Routing:
- net 3.3V: track 0.00 -> 217.9 mm
- net Enc1_2: track 0.00 -> 66.7 mm
- net In4: track 0.00 -> 63.9 mm
- net Enc1_1: track 0.00 -> 63.9 mm
- net PWM2: track 0.00 -> 62.7 mm
- net Output2_1: track 0.00 -> 61.2 mm
- net Output1_1: track 0.00 -> 60.8 mm
- net Output2_2: track 0.00 -> 59.2 mm
- net In3: track 0.00 -> 58.3 mm
- net Output1_2: track 0.00 -> 57.2 mm
- net Enc2_2: track 0.00 -> 55.5 mm
- net Enc2_1: track 0.00 -> 49.5 mm
- net In2: track 0.00 -> 48.7 mm
- net In1: track 0.00 -> 45.1 mm
- net moto_2_state: track 0.00 -> 42.8 mm
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- added copper zone on B.Cu, net 12V
- added copper zone on B.Cu, net 3.3V
- added copper zone on B.Cu, net GND
Other:
- board size 152.4 x 99.1 mm -> 116 x 101 mm
