File: JGA25-370B_with_l289_driver_2_channel.kicad_sch (KiCad schematic)
At the start: 36 parts, among them J1 Power 12 V, J2 Output 1, J3 Encoder 1, J4 Encoder 1 Power 3.3V, J5 Output 2, J6 Encoder 2, J7 Encoder 2 Power 3.3V, J8 Power 5 V, Q1 2N7002, Q2 2N7002, Q3 2N7002, SW1 forward_device_1, SW2 backward_device_1, SW3 stop_device_1, SW4 forward_device_2, SW5 backward_device_2, SW6 stop_device_2, SW7 to_reset_all, U1 L289N_shield, U2 ESP32-S2-DevKitM

Commit message: fix nets
Parts:
- removed J8: Power 5 V, Connector_JST:JST_EH_B2B-EH-A_1x02_P2.50mm_Vertical, symbol Connector:Conn_01x02_Socket
- removed SW7: to_reset_all, Button_Switch_THT:SW_PUSH_6mm_H4.3mm, symbol Switch:SW_Push
- removed U2: ESP32-S2-DevKitM, PCM_Espressif:ESP32-S2-DevKitM, symbol PCM_Espressif:ESP32-S2-DevKitM
- added C1, C2, C8, C9: C, Capacitor_SMD:C_1206_3216Metric, symbol Device:C
- added C10, C3, C7: C_Polarized, Capacitor_THT:CP_Radial_D10.0mm_P2.50mm, symbol Device:C_Polarized
- added C4: ${SIM.PARAMS}, Capacitor_THT:CP_Radial_D10.0mm_P2.50mm, symbol Device:C_Polarized
- added C5, C6: C, Capacitor_THT:C_Disc_D9.0mm_W5.0mm_P5.00mm, symbol Device:C
- added R14: 10k, Resistor_SMD:R_1206_3216Metric, symbol Device:R
- added U2: ESP32-DevKitC, PCM_Espressif:ESP32-DevKitC, symbol PCM_Espressif:ESP32-DevKitC
- added U3: LM1117T-5.0, Package_TO_SOT_THT:TO-220-3_Vertical, symbol Regulator_Linear:LM1117T-5.0
- added U4: LM1117T-3.3, Package_TO_SOT_THT:TO-220-3_Vertical, symbol Regulator_Linear:LM1117T-3.3
- R4, R6: value 330 -> 4.7k
- R5, R8, R9: value 330 -> 10k
- R7: value 330 -> 2.2k
Connections:
- net 12V: now also C1.1, C4.1, C7.1, C8.1, U3.3 (VI), U4.3 (VI)
- net 3.3V: now also SW1.1, SW2.1, SW3.1, SW4.1, SW5.1, SW6.1, C10.1, C9.1, U2.19 (5V), U4.2 (VO)
- net 5V: now also C2.1, C3.1, U2.1 (3V3), U3.2 (VO)
- net Enc1_1: now also U2.28 (GPIO17)
- net Enc1_2: now also U2.27 (GPIO16)
- net Enc2_1: now also U2.15 (MTCK/GPIO13/ADC2_CH4)
- net Enc2_2: now also U2.12 (MTMS/GPIO14/ADC2_CH6)
- net GND: now also R8.2, C1.2, C10.2, C2.2, C3.2, C4.2, C7.2, C8.2, C9.2, R14.2, U2.14 (GND), U2.32 (GND), U2.38 (GND), U3.1 (GND), U4.1 (GND); no longer SW1.2, SW2.2, SW3.2, SW4.2, SW5.2, SW6.2
- net In1: now also U2.36 (GPIO22)
- net In2: now also U2.33 (GPIO21)
- net In3: now also U2.31 (GPIO19)
- net In4: now also U2.30 (GPIO18)
- net Output1_1: now also C6.1
- net Output1_2: now also C6.2
- net Output2_1: now also C5.1
- net Output2_2: now also C5.2
- net PWM1: now also U2.37 (GPIO23)
- net PWM2: now also U2.26 (ADC2_CH0/GPIO4)
- net moto_2_state: now also U2.11 (ADC2_CH7/GPIO27)
- net motor_1_state: now also U2.10 (DAC_2/ADC2_CH9/GPIO26)
- net wifi_state: now also U2.9 (DAC_1/ADC2_CH8/GPIO25)
- net reset: no longer names the net of R6.2
- net reset: now also SW5.2
- net sw_back_1: no longer names the net of R4.2
- net sw_back_1: now also SW2.2; no longer SW2.1
- net sw_back_2 renamed control_curtains_2
- net control_curtains_2: now also R4.1, R7.2, R8.1, U2.8 (32K_XN/GPIO33/ADC1_CH5); no longer SW5.1
- removed net sw_forw_1: R7.2, SW1.1
- removed net sw_forw_2: R8.2, SW4.1
- net sw_stop_1 renamed control_curtains_1
- net control_curtains_1: now also R10.2, R6.1, R14.1, U2.7 (32K_XP/GPIO32/ADC1_CH4); no longer SW3.1
- removed net sw_stop_2: R10.2, SW6.1
- new net: R5.1, SW4.2
- new net: R7.1, SW3.2
- new net: R10.1, SW6.2
- new net: R9.1, SW1.2
- no-connect marks 0 -> 17
Other:
- moved on the sheet: D1, D2, D3, J1, J2, J3, J4, J5, J6, J7, Q1, Q2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

Commit message: ready for order
Parts:
- removed C1, C2, C8, C9: C, Capacitor_SMD:C_1206_3216Metric, symbol Device:C
- removed C10, C7: C_Polarized, Capacitor_THT:CP_Radial_D10.0mm_P2.50mm, symbol Device:C_Polarized
- removed J1: Power 12 V, Connector_JST:JST_EH_B2B-EH-A_1x02_P2.50mm_Vertical, symbol Connector:Conn_01x02_Socket
- removed J2: Output 1, Connector_JST:JST_EH_B2B-EH-A_1x02_P2.50mm_Vertical, symbol Connector:Conn_01x02_Socket
- removed J3: Encoder 1, Connector_JST:JST_EH_B2B-EH-A_1x02_P2.50mm_Vertical, symbol Connector:Conn_01x02_Socket
- removed J4: Encoder 1 Power 3.3V, Connector_JST:JST_EH_B2B-EH-A_1x02_P2.50mm_Vertical, symbol Connector:Conn_01x02_Socket
- removed J5: Output 2, Connector_JST:JST_EH_B2B-EH-A_1x02_P2.50mm_Vertical, symbol Connector:Conn_01x02_Socket
- removed J6: Encoder 2, Connector_JST:JST_EH_B2B-EH-A_1x02_P2.50mm_Vertical, symbol Connector:Conn_01x02_Socket
- removed J7: Encoder 2 Power 3.3V, Connector_JST:JST_EH_B2B-EH-A_1x02_P2.50mm_Vertical, symbol Connector:Conn_01x02_Socket
- removed U3: LM1117T-5.0, Package_TO_SOT_THT:TO-220-3_Vertical, symbol Regulator_Linear:LM1117T-5.0
- removed U4: LM1117T-3.3, Package_TO_SOT_THT:TO-220-3_Vertical, symbol Regulator_Linear:LM1117T-3.3
- added J1, J2, J3, J4: Conn_01x03, TerminalBlock_MetzConnect:TerminalBlock_MetzConnect_Type101_RT01603HBWC_1x03_P5.08mm_Horizontal, symbol Connector_Generic:Conn_01x03
- added J5, J6: Conn_01x04_Pin, Connector_PinHeader_2.54mm:PinHeader_1x04_P2.54mm_Vertical, symbol Connector:Conn_01x04_Pin
- added PS1: Step_Down_3.3v_3A, Converter_DCDC:Converter_DCDC_3A_step_down_3.3v, symbol Converter_DCDC:Converter_DCDC_3A_step_down_3.3v
- renumbered C6 to C1, C5 to C2, D3 to D2, D2 to D3, Q3 to Q2, Q2 to Q3, R2 to R1, R6 to R10, R10 to R11, R14 to R12, R3 to R13, R11 to R14, R9 to R2, R4 to R3, R7 to R4, R8 to R5, R1 to R6, R12 to R7, R13 to R8, R5 to R9, U2 to U1, U1 to U2
Connections:
- net 5V is gone; now on net 3.3V: C3.1, U1.1 (3V3)
- net 12V: now also J2.1 (Pin_1), PS1.1 (+Vin)
- net 3.3V: now also D1.2 (A), D2.2 (A), D3.2 (A), J4.3 (Pin_3), J5.1 (Pin_1), J6.1 (Pin_1), PS1.3 (+Vout); no longer U1.19 (5V)
- net Enc1_1: now also U1.26 (ADC2_CH0/GPIO4), J3.2 (Pin_2), J6.2 (Pin_2); no longer U1.28 (GPIO17)
- net Enc1_2: now also J3.3 (Pin_3), J6.3 (Pin_3)
- net Enc2_1: now also J4.2 (Pin_2)
- net Enc2_2: now also J4.1 (Pin_1)
- net GND: now also R14.2, R6.2, R8.2, J1.3 (Pin_3), J3.1 (Pin_1), J5.4 (Pin_4), J6.4 (Pin_4), PS1.2 (NC), PS1.4 (-Vout); no longer D1.1 (K), D2.1 (K), D3.1 (K)
- net In1: now also U1.30 (GPIO18); no longer U1.36 (GPIO22)
- net In2: now also U1.31 (GPIO19); no longer U1.33 (GPIO21)
- net In3: now also U1.33 (GPIO21), J5.2 (Pin_2); no longer U1.31 (GPIO19)
- net In4: now also U1.36 (GPIO22), J5.3 (Pin_3); no longer U1.30 (GPIO18)
- net Output1_1: now also J1.2 (Pin_2)
- net Output1_2: now also J1.1 (Pin_1)
- net Output2_1: now also J2.3 (Pin_3)
- net Output2_2: now also J2.2 (Pin_2)
- net PWM1: now also U1.28 (GPIO17); no longer U1.37 (GPIO23)
- net PWM2: now also U1.37 (GPIO23); no longer U1.26 (ADC2_CH0/GPIO4)
- net control_curtains_1: now also U1.8 (32K_XN/GPIO33/ADC1_CH5); no longer U1.7 (32K_XP/GPIO32/ADC1_CH4)
- net control_curtains_2: now also U1.7 (32K_XP/GPIO32/ADC1_CH4); no longer U1.8 (32K_XN/GPIO33/ADC1_CH5)
- net at Q2.2 (S): now also R8.1; no longer D2.2 (A)
- net at Q2.3 (D): now also D2.1 (K); no longer R8.2
- net at Q3.2 (S): now also R14.1; no longer D3.2 (A)
- net at Q3.3 (D): now also D3.1 (K); no longer R14.2
- net at Q1.2 (S): now also R6.1; no longer D1.2 (A)
- net at Q1.3 (D): now also D1.1 (K); no longer R6.2
Other:
- moved on the sheet: C1, C2, C3, C4, D1, D2, D3, R14, R6, R8, U2
